File: examples/feather-budget/ecad/sch/Debugger.kicad_sch (KiCad schematic)
At the start: 29 parts, among them J3 USB_C_Receptacle_USB2.0_16P, J8 Conn_ARM_SWD_TagConnect_TC203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, U3 TPD3E001DRLR, U5 nRF52833-QDXX, U6 TXB0106RGY, Y2 32MHz

Commit message: Feather budget example: power, cost and part count judged from KiCad
The seven active parts of the Feather gain hidden, illustrative Power and
Price symbol fields (listed in ecad/NOTICE), and the Model gains power,
cost and part-count requirements whose Model Values are the pre-design
estimates. The recorded netlist fixture is re-recorded with real
kicad-cli 10.0.7, and a real-KiCad test reads the count and both sums.
The requirement defs' short names become two letters, since <'W'>
shadowed SI's watt. docs/engineering-tools.md describes the KiCad adapter
as built.

Users of sysml-viewer check on the example now see the Power and Price
lines with their uncounted parts, and the ComponentCount line.

Co-Authored-By: Claude Opus 5.5 <noreply@anthropic.com>
Parts:
- U5: Power (none) -> 15 mW; Price (none) -> 3.10
- Y2: Power (none) -> 2uW; Price (none) -> 0.30
Changed lines of the file:
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@@
+			)
+		)
+		(property "Power" "15 mW"
+			(at 185.42 93.98 0)
+			(effects
+				(font
+					(size 1.27 1.27)
+				)
+				(hide yes)
+			)
+		)
+		(property "Price" "3.10"
+			(at 185.42 93.98 0)
+			(effects
+				(font
+					(size 1.27 1.27)
+				)
+				(hide yes)
 			)
 		)
@@
 			(effects
 				(font
+					(size 1.27 1.27)
+				)
+				(hide yes)
+			)
+		)
+		(property "Power" "2uW"
+			(at 144.78 63.5 0)
+			(effects
+				(font
+					(size 1.27 1.27)
+				)
+				(hide yes)
+			)
+		)
+		(property "Price" "0.30"
+			(at 144.78 63.5 0)
+			(effects
+				(font
