File: examples/feather-budget/ecad/sch/nPM1300.kicad_sch (KiCad schematic)
At the start: 13 parts, among them U2 nPM1300-QEXX

Commit message: Feather budget example: power, cost and part count judged from KiCad
The seven active parts of the Feather gain hidden, illustrative Power and
Price symbol fields (listed in ecad/NOTICE), and the Model gains power,
cost and part-count requirements whose Model Values are the pre-design
estimates. The recorded netlist fixture is re-recorded with real
kicad-cli 10.0.7, and a real-KiCad test reads the count and both sums.
The requirement defs' short names become two letters, since <'W'>
shadowed SI's watt. docs/engineering-tools.md describes the KiCad adapter
as built.

Users of sysml-viewer check on the example now see the Power and Price
lines with their uncounted parts, and the ComponentCount line.

Co-Authored-By: Claude Opus 5.5 <noreply@anthropic.com>
Parts:
- D3: Power (none) -> 0.03W; Price (none) -> 0.25
- U2: Power (none) -> 350µW; Price (none) -> 2.40
Changed lines of the file:
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@@
+			)
+		)
+		(property "Power" "0.03W"
+			(at 93.98 88.9 0)
+			(effects
+				(font
+					(size 1.27 1.27)
+				)
+				(hide yes)
+			)
+		)
+		(property "Price" "0.25"
+			(at 93.98 88.9 0)
+			(effects
+				(font
+					(size 1.27 1.27)
+				)
+				(hide yes)
 			)
 		)
@@
 			(at 148.59 99.06 0)
 			(effects
+				(font
+					(size 1.27 1.27)
+				)
+				(hide yes)
+			)
+		)
+		(property "Power" "350µW"
+			(at 148.59 99.06 0)
+			(effects
+				(font
+					(size 1.27 1.27)
+				)
+				(hide yes)
+			)
+		)
+		(property "Price" "2.40"
+			(at 148.59 99.06 0)
+			(effects
