File: examples/feather-budget/ecad/sch/nRF54L15.kicad_sch (KiCad schematic)
At the start: 20 parts, among them J6 Conn_01x05_MountingPin, SW1 SW_Push, SW2 SW_Push, U1 BM15x, U4 W25Q16JVUXIQ, Y1 32.768KHz

Commit message: Feather budget example: power, cost and part count judged from KiCad
The seven active parts of the Feather gain hidden, illustrative Power and
Price symbol fields (listed in ecad/NOTICE), and the Model gains power,
cost and part-count requirements whose Model Values are the pre-design
estimates. The recorded netlist fixture is re-recorded with real
kicad-cli 10.0.7, and a real-KiCad test reads the count and both sums.
The requirement defs' short names become two letters, since <'W'>
shadowed SI's watt. docs/engineering-tools.md describes the KiCad adapter
as built.

Users of sysml-viewer check on the example now see the Power and Price
lines with their uncounted parts, and the ComponentCount line.

Co-Authored-By: Claude Opus 5.5 <noreply@anthropic.com>
Parts:
- D1: Power (none) -> 6mW; Price (none) -> 0.05
- U1: Power (none) -> 9.6mW; Price (none) -> 6.50
- Y1: Power (none) -> 1uW; Price (none) -> 0.20
Changed lines of the file:
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@@
+			)
+		)
+		(property "Power" "6mW"
+			(at 93.98 115.57 0)
+			(effects
+				(font
+					(size 1.27 1.27)
+				)
+				(hide yes)
+			)
+		)
+		(property "Price" "0.05"
+			(at 93.98 115.57 0)
+			(effects
+				(font
+					(size 1.27 1.27)
+				)
+				(hide yes)
 			)
 		)
@@
 			)
 		)
+		(property "Power" "1uW"
+			(at 107.95 57.15 0)
+			(effects
+				(font
+					(size 1.27 1.27)
+				)
+				(hide yes)
+			)
+		)
+		(property "Price" "0.20"
+			(at 107.95 57.15 0)
+			(effects
+				(font
+					(size 1.27 1.27)
+				)
+				(hide yes)
+			)
+		)
 		(pin "2"
 		)
@@
 			(at 137.16 90.17 0)
 			(effects
+				(font
+					(size 1.27 1.27)
+				)
+				(hide yes)
+			)
+		)
+		(property "Power" "9.6mW"
+			(at 137.16 90.17 0)
+			(effects
+				(font
+					(size 1.27 1.27)
+				)
+				(hide yes)
+			)
+		)
+		(property "Price" "6.50"
+			(at 137.16 90.17 0)
+			(effects
